File: hardware/Touchstone.sch (EAGLE design)
At the start: 77 parts, among them J3 USB-MICROB, U1 NEOPIXEL_NANO_2427, U10 TSL2591, U11 915MHz, U12 MH-Z19, U13 CCS811-I2C, U14 IAQ-CORE-C, U15 VLP-450-F, U16 VLP-450-F, U2 FT231XQ-R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

Commit message: Updated BOM
MPN added for all parts
Parts:
- C10: MPN (none) -> GRM155R60J475ME47D
- C11, C12, C13, C15, C16, C17, C19, C20, C3, C5, C6, C7, C8: MPN (none) -> GRM155R71C104KA88J
- C14, C18, C2: MPN (none) -> GRM155R60J105KE19D
- C21: MPN (none) -> GRM1555C1H101JA01D
- D1: MPN (none) -> SD103AW-13-F
- R1, R10, R13, R16, R2, R21, R5, R6, R7: MPN (none) -> RC0402FR-0710KL
- R11, R15: MPN (none) -> RC0402JR-0727RL
- R12, R14, R9: MPN (none) -> RC0402FR-07100KL
- R17, R18, R4: MPN (none) -> RC0402FR-07470RL
- R19, R20: MPN (none) -> RC0402JR-071KL
- S1: MPN (none) -> RS-032G05A3-SM RT
- U$4, U$5: MPN (none) -> 0878980426
- U$6: MPN (none) -> M50-3630442
- U1: MPN (none) -> SK6805-2427; PROD_ID (none) -> 3484
- U11: MPN (none) -> RFM69HCW
- U13: MPN (none) -> CCS811
- U14: MPN (none) -> IAQ-CORE C
- U15: MPN (none) -> VLP-550-F
- U16: MPN (none) -> VLP-650-F
- U2: MPN (none) -> FT231XQ-R
- U4: MPN (none) -> Si7021-A20-GM1
- U5: MPN (none) -> ATMEGA328P-MU
- U7: MPN (none) -> 20021311-00010T4LF
- U8: MPN MCP1703T-2502E/CB -> MCP1703T-3302E/CB
- X1: MPN (none) -> CSTCE16M0V53-R0
