File: hardware/Touchstone.brd (EAGLE design)
At the start: 50.8 x 50.8 mm, 77 parts, among them J3 USB-MICROB, U1 NEOPIXEL_NANO_2427, U10 TSL2591, U11 915MHz, U12 MH-Z19, U13 CCS811-I2C, U14 IAQ-CORE-C, U15 VLP-450-F, U16 VLP-450-F, U2 FT231XQ-R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

Commit message: v0.5.7 - updated sound level circuit
- Replaced MEMS mic with mini electret mic
- Added analog circuitry for the mic
- Some routing and silkscreen adjustments
Parts:
- removed C10: 4.7uF, Adafruit Feather 32u4 Bluefruit LE:MICROBUILDER__0402MP
- removed C13: 0.1uF, Adafruit Feather 32u4 Bluefruit LE:MICROBUILDER__0402MP
- removed C14: 1uF, Adafruit Feather 32u4 Bluefruit LE:MICROBUILDER__0402MP
- removed C21: 100pF, Adafruit Feather 32u4 Bluefruit LE:MICROBUILDER__0402MP
- removed R1, R2: 10K, Adafruit Feather 32u4 Bluefruit LE:MICROBUILDER__0402MP
- removed R3: 1.5K, SparkFun-Passives:0805
- removed R8: 100K, SparkFun-Passives:0805
- removed U3: OPA344, SparkFun-AnalogIC:SOT23-5
- removed U6: ADMP401, SparkFun-Sensors:ADMP401
- added C22, C9: 10uF, Adafruit Feather 32u4 Bluefruit LE:MICROBUILDER__0402MP
- added C23, C24: 1uF, Adafruit Feather 32u4 Bluefruit LE:MICROBUILDER__0402MP
- added D3, D4: 120mA/40V/370mV, SparkFun-DiscreteSemi:SOD-523
- added MK1: MIC2-PTH, CMC-4015-40P:MICROPHONE-PTH-4.0MM
- added R22, R27: 1K, Adafruit PowerBoost 1000C Rev B:MICROBUILDER__0402MP
- added R23: 2.2K, Adafruit PowerBoost 1000C Rev B:MICROBUILDER__0402MP
- added R24: 470K, Adafruit PowerBoost 1000C Rev B:MICROBUILDER__0402MP
- added R25, R32: 100, Adafruit PowerBoost 1000C Rev B:MICROBUILDER__0402MP
- added R26, R28, R29, R30: 10K, Adafruit PowerBoost 1000C Rev B:MICROBUILDER__0402MP
- added R31: 22K, Adafruit PowerBoost 1000C Rev B:MICROBUILDER__0402MP
- added U17: LMV324QT, LMV324:QFN-16_3X3
Connections:
- removed net N$10: C21.1, R3.1, R8.2, U3.4
- removed net N$11: C14.1, R1.1, R2.2, U3.3
- removed net OUT: C10.2, U6.1
- new net AMP: C24.1, R24.2, U17.15
- new net N$12: R22.2, R24.1, U17.16
- new net N$14: D3.C, D4.C, R25.1, R31.1
- new net N$15: R27.2, U17.8
- new net N$19: C24.2, R30.2
- new net N$20: C22.2, R25.2, R26.2, U17.9
- new net N$21: D4.A, U17.6
- new net N$22: D3.A, R30.1, R31.2, U17.5
- new net N$8: C9.2, R22.1
- new net VCC/2: R28.2, R29.1, U17.1
- new net _OUT: R27.1, R32.2, U17.7
- net A0: now also R32.1; no longer C21.2, R8.1, U3.1
- net GND: now also C22.1, C23.1, MK1.GND, R26.1, R28.1, U17.11, U17.4; no longer C13.1, C14.2, R2.1, U3.2, U6.2, U6.4, U6.6
- net N$9: now also C9.1, MK1.OUT, R23.1; no longer C10.1, R3.2
- net VCC: now also C23.2, R23.2, R29.2, U17.2; no longer C13.2, R1.2, U3.5, U6.5
Routing:
- net _OUT: track 0.00 -> 26.6 mm, vias 0 -> 3
- net A0: track 29.3 -> 12.5 mm
- net N$20: track 0.00 -> 16.2 mm, vias 0 -> 2
- net N$19: track 0.00 -> 9.24 mm, vias 0 -> 2
- net N$15: track 0.00 -> 8.57 mm, vias 0 -> 2
- net N$10: track 7.19 -> 0.00 mm
- net N$12: track 0.00 -> 6.77 mm
- net N$14: track 0.00 -> 5.40 mm
- net N$22: track 0.00 -> 5.38 mm
- net VCC/2: track 0.00 -> 4.67 mm
- net N$11: track 3.85 -> 0.00 mm
- net VCC: track 241.3 -> 244.9 mm, vias 10 -> 12
- net AMP: track 0.00 -> 3.00 mm
- net N$21: track 0.00 -> 2.28 mm
- net N$9: track 1.94 -> 3.95 mm
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Other:
- board text added: "v0.5.7 | September 2017"
- board text removed: "v0.5.7 | August 2017"
