File: hardware/Touchstone.brd (EAGLE design)
At the start: 50.8 x 50.8 mm, 86 parts, among them J3 USB-MICROB, U1 NEOPIXEL_NANO_2427, U10 TSL2591, U11 915MHz, U12 MH-Z19, U13 CCS811-I2C, U14 IAQ-CORE-C, U15 VLP-450-F, U16 VLP-450-F, U17 LMV324QT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

Commit message: Bug fixes
- Removed pullup from WAKE pin of CSS811 (stopped chip from working)
- Adjusted value of resistor on sound circuit to 1M (to increase gain to
a LOT)
- Minor trace and silkscreen adjustments
- BOM update
Parts:
- removed R14: 100K, Adafruit Feather 32u4 Bluefruit LE:MICROBUILDER__0402MP
- R24: value 470K -> 1M
Connections:
- net D5: no longer R14.2
- net VCC: no longer R14.1
Routing:
- net D5: track 52.7 -> 47.2 mm, vias 3 -> 2
- net VCC: track 244.9 -> 243.1 mm
Other:
- board text added: "v0.5.7 | October 2017"
- board text removed: "v0.5.7 | September 2017"
Changed lines of the file:
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@@
 <text x="9.525" y="23.0632" size="1.016" layer="122" font="vector" ratio="16" rot="MR90" align="center-right">Touchstone</text>
 <text x="30.9372" y="49.5046" size="0.6096" layer="122" font="vector" rot="MR0">Designed by Akram Ali</text>
-<text x="7.9502" y="23.0632" size="0.6096" layer="122" font="vector" rot="MR90" align="center-right">v0.5.7 | September 2017</text>
+<text x="7.9502" y="23.0632" size="0.6096" layer="122" font="vector" rot="MR90" align="center-right">v0.5.7 | October 2017</text>
 <text x="6.7818" y="23.0632" size="0.8128" layer="122" font="vector" ratio="12" rot="MR270" align="center-left">crtlabs.org</text>
 <rectangle x1="1.6002" y1="16.764" x2="2.0066" y2="16.8148" layer="122" rot="R90"/>
@@
 <attribute name="NAME" x="33.782" y="2.8385" size="0.6096" layer="121" font="vector" align="bottom-center"/>
 </element>
-<element name="R14" library="Adafruit Feather 32u4 Bluefruit LE" package="MICROBUILDER__0402MP" value="100K" x="31.6484" y="2.3622" smashed="yes" rot="R180">
-<attribute name="MPN" value="RC0402FR-07100KL" x="31.6484" y="2.3622" size="1.778" layer="27" rot="R180" display="off"/>
-<attribute name="NAME" x="31.7246" y="3.4607" size="0.6096" layer="121" font="vector" rot="R180" align="bottom-center"/>
-</element>
 <element name="U$6" library="CONN_HDR_1.27MM_SMD_4POS" package="CONN_HDR_1.27MM_SMD_4POS" value="CONN_HDR_1.27MM_SMD_4POS" x="45.2882" y="43.1038">
 <attribute name="MPN" value="M50-3630442" x="45.2882" y="43.1038" size="1.778" layer="27" display="off"/>
@@
 <attribute name="NAME" x="47.7203" y="38.6842" size="0.6096" layer="121" font="vector" rot="R270"/>
 </element>
-<element name="R24" library="Adafruit PowerBoost 1000C Rev B" package="MICROBUILDER__0402MP" value="470K" x="42.672" y="33.0708" smashed="yes">
-<attribute name="MPN" value="RC0402JR-07470KL" x="42.672" y="33.0708" size="1.778" layer="27" display="off"/>
+<element name="R24" library="Adafruit PowerBoost 1000C Rev B" package="MICROBUILDER__0402MP" value="1M" x="42.672" y="33.0708" smashed="yes">
+<attribute name="MPN" value="RC0402FR-071ML" x="42.672" y="33.0708" size="1.778" layer="27" display="off"/>
 <attribute name="NAME" x="41.9862" y="33.5979" size="0.6096" layer="121" font="vector"/>
 </element>
@@
 <wire x1="34.814" y1="19.5232" x2="34.4478" y2="19.157" width="0.4064" layer="1"/>
 <contactref element="R12" pad="1"/>
-<contactref element="R14" pad="1"/>
 <via x="35.4076" y="2.5654" extent="1-16" drill="0.25"/>
 <wire x1="35.4076" y1="2.5654" x2="42.1386" y2="2.5654" width="0.1778" layer="16"/>
 <wire x1="42.1386" y1="2.5654" x2="43.3324" y2="3.7592" width="0.1778" layer="16"/>
-<wire x1="32.196759375" y1="2.3622" x2="33.1978" y2="2.3622" width="0.1778" layer="1"/>
-<wire x1="32.196759375" y1="2.3622" x2="32.1564" y2="2.3622" width="0.1778" layer="1"/>
 <wire x1="35.4076" y1="2.5654" x2="35.3568" y2="2.5654" width="0.1778" layer="1"/>
-<wire x1="35.3568" y1="2.5654" x2="34.925" y2="2.9972" width="0.1778" layer="1"/>
-<wire x1="32.831759375" y1="2.9972" x2="32.196759375" y2="2.3622" width="0.1778" layer="1"/>
-<wire x1="34.925" y1="2.9972" x2="32.831759375" y2="2.9972" width="0.1778" layer="1"/>
+<wire x1="34.925" y1="2.9972" x2="35.3568" y2="2.5654" width="0.1778" layer="1"/>
 <wire x1="39.8944" y1="3.4634" x2="39.3614" y2="3.4634" width="0.4064" layer="1"/>
 <wire x1="41.1226" y1="3.2004" x2="40.1574" y2="3.2004" width="0.4064" layer="1"/>
@@
 <wire x1="38.7644" y1="30.2728" x2="38.7604" y2="30.2768" width="0.3048" layer="1"/>
 <via x="38.7604" y="30.2768" extent="1-16" drill="0.25"/>
+<wire x1="33.1978" y1="2.3622" x2="33.1978" y2="2.667" width="0.1778" layer="1"/>
+<wire x1="33.1978" y1="2.667" x2="33.528" y2="2.9972" width="0.1778" layer="1"/>
+<wire x1="33.528" y1="2.9972" x2="34.925" y2="2.9972" width="0.1778" layer="1"/>
 </signal>
 <signal name="SCL">
@@
 <wire x1="38.7614" y1="4.317" x2="38.6588" y2="4.4196" width="0.1778" layer="1"/>
 <via x="38.6588" y="4.4196" extent="1-16" drill="0.25"/>
-<wire x1="38.6588" y1="4.4196" x2="29.792928125" y2="4.4196" width="0.1778" layer="16"/>
+<wire x1="38.6588" y1="4.4196" x2="28.7782" y2="4.4196" width="0.1778" layer="16"/>
 <via x="22.1488" y="27.1272" extent="1-16" drill="0.25"/>
-<contactref element="R14" pad="2"/>
-<wire x1="31.1404" y1="1.7272" x2="30.3276" y2="0.9144" width="0.1778" layer="1"/>
-<via x="30.3276" y="0.9144" extent="1-16" drill="0.25"/>
-<wire x1="30.3276" y1="0.9144" x2="30.3276" y2="3.884928125" width="0.1778" layer="16"/>
-<wire x1="30.3276" y1="3.884928125" x2="29.792928125" y2="4.4196" width="0.1778" layer="16"/>
-<wire x1="31.1404" y1="2.3622" x2="31.1404" y2="1.7272" width="0.1778" layer="1"/>
 <wire x1="38.7614" y1="3.4634" x2="38.7614" y2="4.317" width="0.1778" layer="1"/>
 <wire x1="28.7782" y1="4.4196" x2="28.2194" y2="4.9784" width="0.1778" layer="16"/>
@@
 <wire x1="26.7208" y1="7.8486" x2="25.4254" y2="7.8486" width="0.1778" layer="16"/>
 <wire x1="25.4254" y1="7.8486" x2="24.6126" y2="8.6614" width="0.1778" layer="16"/>
-<wire x1="29.792928125" y1="4.4196" x2="28.7782" y2="4.4196" width="0.1778" layer="16"/>
 <wire x1="24.6126" y1="8.6614" x2="24.6126" y2="12.9032" width="0.1778" layer="16"/>
 <wire x1="24.6126" y1="12.9032" x2="28.4734" y2="16.764" width="0.1778" layer="16"/>

Commit message: PCB adjustments
- Aligned a reistor properly
- Removed some GND vias from underneath the MCU (paste was leaking
through)
Parts:
- moved R12 0.55 mm to (34.2, 2.16), turned to 270 degrees
Routing:
- net VCC: track 243.1 -> 241.5 mm
- net N$6: track 5.14 -> 4.50 mm
- net GND: vias 63 -> 60
Changed lines of the file:
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@@
 <attribute name="MPN" value="0878980426" x="6.477" y="6.7818" size="1.778" layer="27" display="off"/>
 </element>
-<element name="R12" library="Adafruit Feather 32u4 Bluefruit LE" package="MICROBUILDER__0402MP" value="100K" x="33.7058" y="2.3622" smashed="yes">
-<attribute name="MPN" value="RC0402FR-07100KL" x="33.7058" y="2.3622" size="1.778" layer="27" display="off"/>
-<attribute name="NAME" x="33.782" y="2.8385" size="0.6096" layer="121" font="vector" align="bottom-center"/>
+<element name="R12" library="Adafruit Feather 32u4 Bluefruit LE" package="MICROBUILDER__0402MP" value="100K" x="34.2138" y="2.159" smashed="yes" rot="R270">
+<attribute name="MPN" value="RC0402FR-07100KL" x="34.2138" y="2.159" size="1.778" layer="27" rot="R270" display="off"/>
+<attribute name="NAME" x="34.2392" y="3.3465" size="0.6096" layer="121" font="vector" align="bottom-center"/>
 </element>
 <element name="U$6" library="CONN_HDR_1.27MM_SMD_4POS" package="CONN_HDR_1.27MM_SMD_4POS" value="CONN_HDR_1.27MM_SMD_4POS" x="45.2882" y="43.1038">
@@
 <via x="12.3698" y="33.1978" extent="1-16" drill="0.25"/>
 <via x="19.2532" y="27.2796" extent="1-16" drill="0.25"/>
-<via x="24.892" y="35.306" extent="1-16" drill="0.25"/>
-<via x="25.908" y="35.306" extent="1-16" drill="0.25"/>
-<via x="25.908" y="34.29" extent="1-16" drill="0.25"/>
-<via x="24.892" y="34.29" extent="1-16" drill="0.25"/>
 <via x="24.13" y="33.528" extent="1-16" drill="0.25"/>
 <via x="26.67" y="33.528" extent="1-16" drill="0.25"/>
@@
 <contactref element="U17" pad="4"/>
 <contactref element="MK1" pad="GND"/>
+<via x="25.4" y="34.798" extent="1-16" drill="0.25"/>
 </signal>
 <signal name="VCC">
@@
 <wire x1="35.4076" y1="2.5654" x2="42.1386" y2="2.5654" width="0.1778" layer="16"/>
 <wire x1="42.1386" y1="2.5654" x2="43.3324" y2="3.7592" width="0.1778" layer="16"/>
-<wire x1="35.4076" y1="2.5654" x2="35.3568" y2="2.5654" width="0.1778" layer="1"/>
-<wire x1="34.925" y1="2.9972" x2="35.3568" y2="2.5654" width="0.1778" layer="1"/>
+<wire x1="35.3568" y1="2.5654" x2="35.4076" y2="2.5654" width="0.1778" layer="1"/>
 <wire x1="39.8944" y1="3.4634" x2="39.3614" y2="3.4634" width="0.4064" layer="1"/>
 <wire x1="41.1226" y1="3.2004" x2="40.1574" y2="3.2004" width="0.4064" layer="1"/>
@@
 <wire x1="38.7644" y1="30.2728" x2="38.7604" y2="30.2768" width="0.3048" layer="1"/>
 <via x="38.7604" y="30.2768" extent="1-16" drill="0.25"/>
-<wire x1="33.1978" y1="2.3622" x2="33.1978" y2="2.667" width="0.1778" layer="1"/>
-<wire x1="33.1978" y1="2.667" x2="33.528" y2="2.9972" width="0.1778" layer="1"/>
-<wire x1="33.528" y1="2.9972" x2="34.925" y2="2.9972" width="0.1778" layer="1"/>
+<wire x1="34.925" y1="2.5654" x2="35.4076" y2="2.5654" width="0.1778" layer="1"/>
+<wire x1="34.2138" y1="2.667" x2="34.8234" y2="2.667" width="0.1778" layer="1"/>
+<wire x1="34.8234" y1="2.667" x2="34.925" y2="2.5654" width="0.1778" layer="1"/>
 </signal>
 <signal name="SCL">
@@
 <wire x1="37.3888" y1="0.5588" x2="37.5614" y2="0.7314" width="0.1778" layer="1"/>
 <wire x1="35.433" y1="0.5588" x2="37.3888" y2="0.5588" width="0.1778" layer="1"/>
-<wire x1="34.2138" y1="1.778" x2="35.433" y2="0.5588" width="0.1778" layer="1"/>
-<wire x1="34.2138" y1="2.3622" x2="34.2138" y2="1.778" width="0.1778" layer="1"/>
 <wire x1="37.5614" y1="0.7314" x2="37.5614" y2="1.3634" width="0.1778" layer="1"/>
+<wire x1="34.2138" y1="1.651" x2="34.3408" y2="1.651" width="0.1778" layer="1"/>
+<wire x1="34.3408" y1="1.651" x2="35.433" y2="0.5588" width="0.1778" layer="1"/>
 </signal>
 <signal name="N$7">

Commit message: Added gerbers and BOM
- Also updated firmware for button interrupt, sound level stuff
Parts:
- R24: value 1M -> 470K
Changed lines of the file:
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@@
 <attribute name="NAME" x="47.7203" y="38.6842" size="0.6096" layer="121" font="vector" rot="R270"/>
 </element>
-<element name="R24" library="Adafruit PowerBoost 1000C Rev B" package="MICROBUILDER__0402MP" value="1M" x="42.672" y="33.0708" smashed="yes">
+<element name="R24" library="Adafruit PowerBoost 1000C Rev B" package="MICROBUILDER__0402MP" value="470K" x="42.672" y="33.0708" smashed="yes">
 <attribute name="MPN" value="RC0402FR-071ML" x="42.672" y="33.0708" size="1.778" layer="27" display="off"/>
 <attribute name="NAME" x="41.9862" y="33.5979" size="0.6096" layer="121" font="vector"/>
